File: top board 3.6.sch (EAGLE design)
At the start: 31 parts

Commit message: began routing
Parts:
- removed C1: 2.2uF, Seeed-OPL-Capacitor:CERAMIC-0.5PF-50V-0.1PF-NPO(0603)
- removed C2: 22uF, Seeed-OPL-Capacitor:CERAMIC-0.5PF-50V-0.1PF-NPO(0603)
- removed C3: 100nF, Seeed-OPL-Capacitor:CERAMIC-1PF-50V-0.25PF-NPO(0603)
- removed C4, C7: 100nF, Seeed-OPL-Capacitor:CERAMIC-0.5PF-50V-0.1PF-NPO(0603)
- removed C5: 10pF, Seeed-OPL-Capacitor:CERAMIC-0.5PF-50V-0.1PF-NPO(0603)
- removed C6: 15pF, Seeed-OPL-Capacitor:CERAMIC-0.5PF-50V-0.1PF-NPO(0603)
- removed C8, C9: 10uF, Seeed-OPL-Capacitor:CERAMIC-0.5PF-50V-0.1PF-NPO(0603)
- removed CLK: FXO_HC73, CUSTOM:FXO_HC73
- removed D1: B130-13-F, CUSTOM:B130-13-F
- removed DRIVER: TB6593FNG, CUSTOM:TB6593FNG
- removed KEY: PTS645, CUSTOM:BUTTON
- removed L1: DFE252012C, CUSTOM:DFE252012C
- removed MDL1: (no value), adafruit:ESP-12
- removed OPAMP: AZV321, Diodes_Inc_By_element14_Batch_1:LMV321SEG-7
- removed R10, R3, R4, R9: 10k, resistor:R-US_R0603
- removed R2, R6: 470, resistor:R-US_R0603
- removed R5: 100k, resistor:R-US_R0603
- removed R7: 285, resistor:R-US_R0603
- removed R8: 1k, resistor:R-US_R0603
- removed SW: RN1906FE, CUSTOM:RN1906FE
- removed U$1: AVX_CONN, CUSTOM:AVX_CONN
- removed U1: (no value), MicroUSB:USB""
- removed UART: CH340G, CUSTOM:CH340G
- added SLIP: RING2, CUSTOM:RING2
- added U$2: AVX_CONN, CUSTOM:AVX_CONN
- R1: value 10k -> 67
- REG: value TPS62177 -> LM334MX; device CUSTOM:TPS62177 -> CUSTOM:LM334MX
Connections:
- removed net +3V3: C2.2, C4.2, C7.2, C8.2, C9.2, DRIVER.VCC, L1.P$2, MDL1.VCC, OPAMP.V+, R1.1, R10.1, R3.1, R4.1, R5.2, REG.SLEEP, REG.VOS, UART.V3, UART.VCC
- removed net ADC: MDL1.ADC, OPAMP.OUT, R7.2
- removed net D+: U1.D+, UART.UD+
- removed net D-: U1.D-, UART.UD-
- removed net DTR: SW.B2, SW.E1, UART.DTR
- removed net EN: MDL1.CH_PD, R3.2
- removed net GP0: MDL1.GPIO0, R1.2, SW.C1
- removed net GP14: MDL1.GPIO14
- removed net GP15: MDL1.GPIO15, R9.2
- removed net GP16: MDL1.GPIO16
- removed net GP2: MDL1.GPIO2, R10.2
- removed net IN1: DRIVER.IN1, MDL1.GPIO13
- removed net IN2: DRIVER.IN2, MDL1.GPIO12
- removed net M1: DRIVER.11, DRIVER.12
- removed net M2: DRIVER.21, DRIVER.22
- removed net N$1: R2.2, UART.TXD
- removed net N$2: R5.1, REG.PG
- removed net N$3: D1.AN, U1.VBUS
- removed net N$4: L1.P$1, REG.SW
- removed net N$5: OPAMP.IN+, U$1.P2
- removed net N$6: OPAMP.IN-, R7.1, R8.2
- removed net N$7: R6.2, UART.RXD
- removed net PWM: DRIVER.PWM, MDL1.GPIO4
- removed net RST: C3.2, KEY.1, MDL1.RESET, R4.2, SW.C2
- removed net RTS: SW.B1, SW.E2, UART.RTS
- removed net RX: MDL1.RXD, R6.1
- removed net STBY: DRIVER.STBY, MDL1.GPIO5
- removed net TX: MDL1.TXD, R2.1
- removed net XI: C5.1, CLK.VDD, UART.XI
- removed net XO: C6.1, CLK.OUT, UART.XO
- new net N$8: R1.2, REG.R
- new net N$9: R1.1, REG.V-, SLIP.D
- net GND: now also SLIP.GND, U$2.P1; no longer C1.1, C2.1, C3.1, C4.1, C5.2, C6.2, C7.1, C8.1, C9.1, CLK.GND, DRIVER.GND, DRIVER.PG1, DRIVER.PG2, DRIVER.PG3, DRIVER.PG4, DRIVER.PG5, DRIVER.PG6, KEY.3, MDL1.GND, OPAMP.V-, R8.1, R9.1, REG.AGND, REG.FB, REG.NC, REG.PAD, REG.PGND, U$1.P3, U1.GND, UART.GND
- net VCC: now also REG.V+, SLIP.V+, U$2.P3; no longer C1.2, D1.CATH, DRIVER.VM1, DRIVER.VM2, DRIVER.VM3, DRIVER.VM4, REG.EN, REG.VIN, U$1.P1
Other:
- moved on the sheet: R1
