File: top board.brd (EAGLE design)
At the start: 60 x 60 mm, 2 parts

Commit message: began routing
Parts:
- removed U$1: AVX_CONN, CUSTOM:AVX_CONN
- added R1: 67, resistor:R0603
- added REG: LM334MX, CUSTOM:8-SOIC
- added SLIP: RING, CUSTOM:RING
- U$2: value RING -> AVX_CONN; device CUSTOM:RING -> CUSTOM:AVX_CONN
- moved U$2 25.0 mm to (30.0, 55.0), flipped to the bottom, turned to 90 degrees
Connections:
- removed net N$3: U$1.P1, U$2.P$2
- removed net N$4: U$1.P3, U$2.P$1
- new net GND: SLIP.GND, U$2.P1
- new net N$8: R1.2, REG.1
- new net N$9: R1.1, REG.2, SLIP.D+
- new net VCC: REG.4, SLIP.V+, U$2.P3
Routing:
- net VCC: track 0.00 -> 96.5 mm, vias 0 -> 2
- net N$9: track 0.00 -> 8.47 mm
- net GND: track 0.00 -> 7.30 mm, vias 0 -> 1
- net N$4: track 7.25 -> 0.00 mm, vias 1 -> 0
- net N$3: track 7.25 -> 0.00 mm, vias 1 -> 0
- net N$8: track 0.00 -> 4.60 mm
