File: top board.sch (EAGLE design)
At the start: 2 parts

Commit message: began routing
Parts:
- removed U$1: AVX_CONN, CUSTOM:AVX_CONN
- added R1: 67, resistor:R-US_R0603
- added REG: LM334MX, CUSTOM:LM334MX
- added SLIP: RING, CUSTOM:RING
- U$2: value RING -> AVX_CONN; device CUSTOM:RING -> CUSTOM:AVX_CONN
Connections:
- removed net N$3: U$1.P1, U$2.P$2
- removed net N$4: U$1.P3, U$2.P$1
- new net GND: SLIP.GND, U$2.P1
- new net N$8: R1.2, REG.R
- new net N$9: R1.1, REG.V-, SLIP.D
- new net VCC: REG.V+, SLIP.V+, U$2.P3
