File: motherboard.brd (EAGLE design)
At the start: 71.1 x 35.6 mm, 33 parts

Commit message: Add files via upload
Final version of gen1 boards, added initial cad of slipring with analog ground, switching to bourns connectors
Parts:
- added C12: 100nF, Seeed-OPL-Capacitor:C0603
- R1: value 10k -> 1k
- R9: value 285 -> 33k
- moved R1 3.38 mm to (54.5, 12.8)
- moved C4 1.63 mm to (60.7, 12.1)
- moved C3 1.47 mm to (62.4, 12.1)
Connections:
- net EN: now also C12.2
- net GND: now also C12.1
Routing:
- net EN: track 2.18 -> 5.99 mm
- net RST: track 62.0 -> 65.4 mm
- net IN2: track 30.4 -> 33.7 mm
- net +3V3: track 133.9 -> 136.8 mm
- net IN1: track 33.3 -> 34.7 mm
