File: motherboard.brd (EAGLE design)
At the start: 71.1 x 35.6 mm, 34 parts

Commit message: more routing
Parts:
- removed U$1: BOURNS_4PIN, CUSTOM:BOURNS_4PIN
- added CONN: BOURNS_2PIN, CUSTOM:BOURNS_2PIN
- added R11, R12: 100, resistor:R0603
- added U$2: BI_LED, CUSTOM:BI_LED
- added U$3: 4PIN_HEADER, CUSTOM:4PIN_HEADER
- added WIPER: BOURNS_4PIN, CUSTOM:BOURNS_4PIN
- KEY: value PTS645 -> PTS810
- R9: value 33k -> 5k
- moved C10 67.0 mm to (7.29, 18.8)
- moved C11 67.0 mm to (5.39, 18.8)
- moved UART 63.7 mm to (14.0, 18.0)
- moved KEY 59.5 mm to (5.00, 12.0), flipped to the bottom
- moved R7 59.1 mm to (11.5, 4.89)
- moved C6 58.1 mm to (9.68, 12.5)
- moved SW 56.9 mm to (20.0, 20.0), turned to 90 degrees
- moved C5 55.1 mm to (10.2, 10.3)
- moved R6 55.0 mm to (14.8, 10.4)
- moved D1 54.7 mm to (37.0, 48.0), turned to 180 degrees
- moved CLK 52.5 mm to (16.0, 11.0), turned to 0 degrees
- moved MICRO-USB 50.3 mm to (32.5, 42.0)
- moved R5 44.6 mm to (27.1, 2.02)
- moved C7 42.8 mm to (63.1, 14.3)
- moved C1 40.8 mm to (46.0, 56.7)
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Connections:
- removed net GP14: ESP12.5
- removed net GP16: ESP12.4
- removed net N$3: D1.AN, MICRO-USB.VCC
- new net N$11: R11.1, U$2.2
- new net N$12: R12.1, U$2.3
- new net N$8: ESP12.5, R12.2
- new net N$9: ESP12.4, R11.2
- new net USB+: D1.AN, MICRO-USB.VCC, U$3.1
- net D+: now also U$3.3
- net D-: now also U$3.2
- net GND: now also CONN.P2, U$2.1, U$2.4, U$3.4, WIPER.P1, WIPER.P2; no longer U$1.P1, U$1.P3
- net N$5: now also WIPER.P4; no longer U$1.P4
- net VCC: now also CONN.P1, WIPER.P3; no longer U$1.P2
Routing:
- net RST: track 67.6 -> 22.5 mm, vias 4 -> 2
- net TX: track 45.0 -> 0.00 mm, vias 2 -> 0
- net +3V3: track 136.8 -> 93.8 mm, vias 7 -> 5
- net RX: track 43.0 -> 0.00 mm, vias 2 -> 0
- net GP0: track 42.7 -> 3.65 mm, vias 2 -> 1
- net XI: track 28.8 -> 0.00 mm, vias 2 -> 0
- net STBY: track 50.9 -> 28.4 mm, vias 2 -> 0
- net PWM: track 52.3 -> 31.6 mm, vias 2 -> 0
- net VCC: track 98.1 -> 80.1 mm, vias 4 -> 3
- net N$5: track 15.7 -> 25.0 mm
- net N$3: track 8.64 -> 0.00 mm
- net ADC: track 25.2 -> 18.0 mm, vias 0 -> 2
- net D-: track 8.10 -> 1.32 mm, vias 2 -> 0
- net N$7: track 6.77 -> 0.00 mm
- net USB+: track 0.00 -> 5.90 mm
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- removed copper zone on layer 1, net +3V3
- removed copper zone on layer 1, net SW
Other:
- board size 71.1 x 35.6 mm -> 61.8 x 64.9 mm
- board text removed: "+"
- board text removed: "-"

Commit message: final routing before splitting up boards
Parts:
- moved KEY 33.0 mm to (38.0, 11.0), turned to 90 degrees
- moved C7 16.6 mm to (46.5, 15.0), turned to 0 degrees
- moved C8 13.8 mm to (47.5, 10.0)
- moved C5 10.3 mm to (19.0, 5.00), turned to 90 degrees
- moved R7 7.26 mm to (10.0, 12.0), turned to 90 degrees
- moved C11 4.94 mm to (10.0, 17.0), flipped to the bottom, turned to 90 degrees
- moved C6 4.35 mm to (14.0, 12.0), turned to 0 degrees
- moved R6 3.25 mm to (12.0, 12.0), turned to 90 degrees
- moved C10 2.72 mm to (10.0, 19.0), flipped to the bottom, turned to 90 degrees
- moved CLK 2.24 mm to (18.0, 10.0), turned to 90 degrees
- moved R2 2.24 mm to (40.0, 18.0), turned to 0 degrees
- moved UART 1.00 mm to (13.0, 18.0)
Connections:
- net GND: now also KEY.4; no longer KEY.3
- net RST: now also KEY.2; no longer KEY.1
Routing:
- net +3V3: track 93.8 -> 134.0 mm, vias 5 -> 7
- net TX: track 0.00 -> 30.5 mm
- net RX: track 0.00 -> 29.9 mm, vias 0 -> 2
- net GP0: track 3.65 -> 28.4 mm, vias 1 -> 4
- net D-: track 1.32 -> 25.8 mm, vias 0 -> 3
- net RTS: track 0.00 -> 15.2 mm
- net D+: track 1.57 -> 16.0 mm, vias 0 -> 3
- net DTR: track 0.00 -> 11.2 mm
- net XI: track 0.00 -> 5.32 mm
- net RST: track 22.5 -> 27.5 mm
- net N$7: track 0.00 -> 2.98 mm
- net N$1: track 0.00 -> 2.68 mm
- net VCC: track 80.1 -> 82.4 mm
- net IN2: track 31.4 -> 30.2 mm
- net IN1: track 34.8 -> 33.5 mm
Other:
- board text added: "3V3"
- board text added: "D+"
- board text added: "D-"
- board text added: "VCC"
