File: motherboard.brd (EAGLE design)
At the start: 61.8 x 64.9 mm, 39 parts

Commit message: Added BOM, updated resistor values
Parts:
- R11, R12: value 100 -> 330
- R9: value 5k -> 5.1k
Changed lines of the file:
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@@
 <element name="KEY" library="CUSTOM" package="BUTTON" value="PTS810" x="38" y="11" rot="MR90"/>
 <element name="D1" library="CUSTOM" package="SMA" value="B130-13-F" x="37" y="48" smashed="yes" rot="R180"/>
-<element name="R9" library="resistor" package="R0603" value="5k" x="44" y="44.6" smashed="yes">
+<element name="R9" library="resistor" package="R0603" value="5.1k" x="44" y="44.6" smashed="yes">
 <attribute name="NAME" x="40.251" y="43.865" size="1.27" layer="25"/>
 <attribute name="VALUE" x="43.365" y="42.695" size="1.27" layer="27"/>
@@
 </element>
 <element name="U$2" library="CUSTOM" package="BI_LED" value="BI_LED" x="26.998" y="12.03" rot="MR90"/>
-<element name="R11" library="resistor" package="R0603" value="100" x="31" y="15" smashed="yes" rot="MR90">
+<element name="R11" library="resistor" package="R0603" value="330" x="31" y="15" smashed="yes" rot="MR90">
 <attribute name="NAME" x="30.435" y="10.265" size="1.27" layer="26" rot="MR90"/>
 <attribute name="VALUE" x="29.095" y="14.365" size="1.27" layer="28" rot="MR90"/>
 </element>
-<element name="R12" library="resistor" package="R0603" value="100" x="29" y="15" smashed="yes" rot="MR90">
+<element name="R12" library="resistor" package="R0603" value="330" x="29" y="15" smashed="yes" rot="MR90">
 <attribute name="NAME" x="26.835" y="14.165" size="1.27" layer="26" rot="MR90"/>
 <attribute name="VALUE" x="27.095" y="14.365" size="1.27" layer="28" rot="MR90"/>
