File: espboard.sch (EAGLE design)
At the start: 26 parts

Commit message: fixed intial board errors, including short, flipped usb, and missing trace
Parts:
- R11, R12: value 100 -> 330
Changed lines of the file:
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@@
 <part name="GND24" library="supply1" deviceset="GND" device=""/>
 <part name="U$2" library="CUSTOM" deviceset="BI_LED" device=""/>
-<part name="R11" library="resistor" deviceset="R-US_" device="R0603" value="100"/>
-<part name="R12" library="resistor" deviceset="R-US_" device="R0603" value="100"/>
+<part name="R11" library="resistor" deviceset="R-US_" device="R0603" value="330"/>
+<part name="R12" library="resistor" deviceset="R-US_" device="R0603" value="330"/>
 <part name="GND26" library="supply1" deviceset="GND" device=""/>
 <part name="GND27" library="supply1" deviceset="GND" device=""/>
