File: wiperboard.sch (EAGLE design)
At the start: 12 parts

Commit message: fixed intial board errors, including short, flipped usb, and missing trace
Connections:
- net D+: now also U$3.2; no longer U$3.3
- net D-: now also U$3.3; no longer U$3.2
- net GND: now also CONN.P3, U$3.1, WIPER.P7, WIPER.P8; no longer U$3.4
- net N$5: now also WIPER.P5
- net USB+: now also U$3.4; no longer U$3.1
- net VCC: now also CONN.P4, WIPER.P6
Other:
- moved on the sheet: AMP, D1, R8, R9
Changed lines of the file:
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@@
 <instance part="FRAME1" gate="G$1" x="0" y="0"/>
 <instance part="FRAME1" gate="G$2" x="172.72" y="0"/>
-<instance part="AMP" gate="A" x="45.72" y="198.12"/>
+<instance part="AMP" gate="A" x="114.3" y="182.88"/>
 <instance part="REG" gate="G$1" x="226.06" y="119.38"/>
 <instance part="P+1" gate="VCC" x="203.2" y="137.16"/>
@@
 <instance part="GND9" gate="1" x="259.08" y="104.14"/>
 <instance part="+3V1" gate="G$1" x="259.08" y="137.16"/>
-<instance part="D1" gate="G$1" x="12.7" y="144.78" rot="R90"/>
-<instance part="P+3" gate="VCC" x="12.7" y="157.48"/>
-<instance part="R9" gate="G$1" x="63.5" y="172.72"/>
-<instance part="R8" gate="G$1" x="35.56" y="172.72"/>
-<instance part="GND15" gate="1" x="27.94" y="167.64"/>
-<instance part="+3V6" gate="G$1" x="43.18" y="205.74"/>
+<instance part="D1" gate="G$1" x="50.8" y="127" rot="R90"/>
+<instance part="P+3" gate="VCC" x="50.8" y="137.16"/>
+<instance part="R9" gate="G$1" x="132.08" y="157.48"/>
+<instance part="R8" gate="G$1" x="104.14" y="157.48"/>
+<instance part="GND15" gate="1" x="96.52" y="152.4"/>
+<instance part="+3V6" gate="G$1" x="111.76" y="190.5"/>
 <instance part="+3V8" gate="G$1" x="210.82" y="137.16"/>
 <instance part="L1" gate="G$1" x="248.92" y="129.54"/>
-<instance part="WIPER" gate="G$1" x="15.24" y="195.58" rot="R180"/>
-<instance part="P+2" gate="VCC" x="30.48" y="208.28"/>
+<instance part="WIPER" gate="G$1" x="83.82" y="180.34" rot="R180"/>
+<instance part="P+2" gate="VCC" x="99.06" y="193.04"/>
 <instance part="U$3" gate="G$1" x="17.78" y="119.38"/>
-<instance part="GND7" gate="1" x="33.02" y="111.76" rot="R90"/>
+<instance part="GND7" gate="1" x="25.4" y="134.62" rot="R180"/>
 <instance part="CONN" gate="G$1" x="139.7" y="30.48"/>
 <instance part="P+5" gate="VCC" x="129.54" y="38.1"/>
@@
 <segment>
 <pinref part="R9" gate="G$1" pin="2"/>
-<wire x1="68.58" y1="172.72" x2="83.82" y2="172.72" width="0.1524" layer="91"/>
-<wire x1="83.82" y1="172.72" x2="83.82" y2="198.12" width="0.1524" layer="91"/>
+<wire x1="137.16" y1="157.48" x2="152.4" y2="157.48" width="0.1524" layer="91"/>
+<wire x1="152.4" y1="157.48" x2="152.4" y2="182.88" width="0.1524" layer="91"/>
 <pinref part="AMP" gate="A" pin="OUT"/>
-<wire x1="83.82" y1="198.12" x2="81.28" y2="198.12" width="0.1524" layer="91"/>
-<wire x1="83.82" y1="198.12" x2="88.9" y2="198.12" width="0.1524" layer="91"/>
-<junction x="83.82" y="198.12"/>
-<label x="83.82" y="198.12" size="1.778" layer="95"/>
+<wire x1="152.4" y1="182.88" x2="149.86" y2="182.88" width="0.1524" layer="91"/>
+<wire x1="152.4" y1="182.88" x2="157.48" y2="182.88" width="0.1524" layer="91"/>
+<junction x="152.4" y="182.88"/>
+<label x="152.4" y="182.88" size="1.778" layer="95"/>
 </segment>
 </net>
@@
 <segment>
 <pinref part="GND15" gate="1" pin="GND"/>
-<wire x1="27.94" y1="170.18" x2="27.94" y2="172.72" width="0.1524" layer="91"/>
+<wire x1="96.52" y1="154.94" x2="96.52" y2="157.48" width="0.1524" layer="91"/>
 <pinref part="R8" gate="G$1" pin="1"/>
-<wire x1="27.94" y1="172.72" x2="30.48" y2="172.72" width="0.1524" layer="91"/>
+<wire x1="96.52" y1="157.48" x2="99.06" y2="157.48" width="0.1524" layer="91"/>
 <pinref part="AMP" gate="A" pin="V-"/>
-<wire x1="45.72" y1="185.42" x2="27.94" y2="185.42" width="0.1524" layer="91"/>
-<wire x1="27.94" y1="185.42" x2="27.94" y2="172.72" width="0.1524" layer="91"/>
-<junction x="27.94" y="172.72"/>
-<junction x="27.94" y="185.42"/>
+<wire x1="114.3" y1="170.18" x2="96.52" y2="170.18" width="0.1524" layer="91"/>
+<wire x1="96.52" y1="170.18" x2="96.52" y2="157.48" width="0.1524" layer="91"/>
+<junction x="96.52" y="157.48"/>
+<junction x="96.52" y="170.18"/>
 <pinref part="WIPER" gate="G$1" pin="P1"/>
-<wire x1="27.94" y1="187.96" x2="27.94" y2="185.42" width="0.1524" layer="91"/>
-<wire x1="25.4" y1="187.96" x2="27.94" y2="187.96" width="0.1524" layer="91"/>
+<wire x1="96.52" y1="172.72" x2="96.52" y2="170.18" width="0.1524" layer="91"/>
+<wire x1="93.98" y1="172.72" x2="96.52" y2="172.72" width="0.1524" layer="91"/>
 <pinref part="WIPER" gate="G$1" pin="P2"/>
-<wire x1="25.4" y1="193.04" x2="27.94" y2="193.04" width="0.1524" layer="91"/>
-<wire x1="27.94" y1="193.04" x2="27.94" y2="187.96" width="0.1524" layer="91"/>
-<junction x="27.94" y="187.96"/>
-</segment>
-<segment>
-<pinref part="U$3" gate="G$1" pin="4"/>
-<wire x1="22.86" y1="111.76" x2="30.48" y2="111.76" width="0.1524" layer="91"/>
-<pinref part="GND7" gate="1" pin="GND"/>
+<wire x1="93.98" y1="177.8" x2="96.52" y2="177.8" width="0.1524" layer="91"/>
+<wire x1="96.52" y1="177.8" x2="96.52" y2="172.72" width="0.1524" layer="91"/>
+<junction x="96.52" y="172.72"/>
+<pinref part="WIPER" gate="G$1" pin="P7"/>
+<wire x1="71.12" y1="177.8" x2="93.98" y2="177.8" width="0.1524" layer="91"/>
+<junction x="93.98" y="177.8"/>
+<pinref part="WIPER" gate="G$1" pin="P8"/>
+<wire x1="93.98" y1="172.72" x2="71.12" y2="172.72" width="0.1524" layer="91"/>
+<junction x="93.98" y="172.72"/>
 </segment>
 <segment>
@@
 <wire x1="132.08" y1="27.94" x2="129.54" y2="27.94" width="0.1524" layer="91"/>
 <wire x1="129.54" y1="27.94" x2="129.54" y2="25.4" width="0.1524" layer="91"/>
+<pinref part="CONN" gate="G$1" pin="P3"/>
+<wire x1="152.4" y1="27.94" x2="132.08" y2="27.94" width="0.1524" layer="91"/>
+<junction x="132.08" y="27.94"/>
+</segment>
+<segment>
+<pinref part="U$3" gate="G$1" pin="1"/>
+<wire x1="22.86" y1="127" x2="25.4" y2="127" width="0.1524" layer="91"/>
+<wire x1="25.4" y1="127" x2="25.4" y2="132.08" width="0.1524" layer="91"/>
+<pinref part="GND7" gate="1" pin="GND"/>
 </segment>
 </net>
@@
 <pinref part="P+3" gate="VCC" pin="VCC"/>
 <pinref part="D1" gate="G$1" pin="CATH"/>
-<wire x1="12.7" y1="154.94" x2="12.7" y2="149.86" width="0.1524" layer="91"/>
+<wire x1="50.8" y1="134.62" x2="50.8" y2="132.08" width="0.1524" layer="91"/>
 </segment>
 <segment>
 <pinref part="WIPER" gate="G$1" pin="P3"/>
 <pinref part="P+2" gate="VCC" pin="VCC"/>
-<wire x1="25.4" y1="198.12" x2="30.48" y2="198.12" width="0.1524" layer="91"/>
-<wire x1="30.48" y1="198.12" x2="30.48" y2="205.74" width="0.1524" layer="91"/>
+<wire x1="93.98" y1="182.88" x2="99.06" y2="182.88" width="0.1524" layer="91"/>
+<wire x1="99.06" y1="182.88" x2="99.06" y2="190.5" width="0.1524" layer="91"/>
+<pinref part="WIPER" gate="G$1" pin="P6"/>
+<wire x1="93.98" y1="182.88" x2="71.12" y2="182.88" width="0.1524" layer="91"/>
+<junction x="93.98" y="182.88"/>
 </segment>
 <segment>
@@
 <wire x1="132.08" y1="33.02" x2="129.54" y2="33.02" width="0.1524" layer="91"/>
 <wire x1="129.54" y1="33.02" x2="129.54" y2="35.56" width="0.1524" layer="91"/>
+<pinref part="CONN" gate="G$1" pin="P4"/>
+<wire x1="132.08" y1="33.02" x2="152.4" y2="33.02" width="0.1524" layer="91"/>
+<junction x="132.08" y="33.02"/>
 </segment>
 </net>
@@
 <segment>
 <pinref part="AMP" gate="A" pin="V+"/>
-<wire x1="45.72" y1="198.12" x2="43.18" y2="198.12" width="0.1524" layer="91"/>
-<wire x1="43.18" y1="198.12" x2="43.18" y2="203.2" width="0.1524" layer="91"/>
+<wire x1="114.3" y1="182.88" x2="111.76" y2="182.88" width="0.1524" layer="91"/>
+<wire x1="111.76" y1="182.88" x2="111.76" y2="187.96" width="0.1524" layer="91"/>
 <pinref part="+3V6" gate="G$1" pin="+3V3"/>
 </segment>
@@
 </segment>
 </net>
-<net name="D+" class="0">
+<net name="D-" class="0">
 <segment>
 <label x="38.1" y="132.08" size="1.778" layer="95"/>
@@
 </segment>
 </net>
-<net name="D-" class="0">
+<net name="D+" class="0">
 <segment>
 <label x="38.1" y="127" size="1.778" layer="95"/>
@@
 <pinref part="AMP" gate="A" pin="IN+"/>
 <pinref part="WIPER" gate="G$1" pin="P4"/>
-<wire x1="25.4" y1="203.2" x2="35.56" y2="203.2" width="0.1524" layer="91"/>
-<wire x1="35.56" y1="203.2" x2="35.56" y2="193.04" width="0.1524" layer="91"/>
-<wire x1="35.56" y1="193.04" x2="45.72" y2="193.04" width="0.1524" layer="91"/>
+<wire x1="93.98" y1="187.96" x2="104.14" y2="187.96" width="0.1524" layer="91"/>
+<wire x1="104.14" y1="187.96" x2="104.14" y2="177.8" width="0.1524" layer="91"/>
+<wire x1="104.14" y1="177.8" x2="114.3" y2="177.8" width="0.1524" layer="91"/>
+<pinref part="WIPER" gate="G$1" pin="P5"/>
+<wire x1="71.12" y1="187.96" x2="93.98" y2="187.96" width="0.1524" layer="91"/>
+<junction x="93.98" y="187.96"/>
 </segment>
 </net>
@@
 <segment>
 <pinref part="AMP" gate="A" pin="IN-"/>
-<wire x1="45.72" y1="190.5" x2="43.18" y2="190.5" width="0.1524" layer="91"/>
-<wire x1="43.18" y1="190.5" x2="43.18" y2="172.72" width="0.1524" layer="91"/>
+<wire x1="114.3" y1="175.26" x2="111.76" y2="175.26" width="0.1524" layer="91"/>
+<wire x1="111.76" y1="175.26" x2="111.76" y2="157.48" width="0.1524" layer="91"/>
 <pinref part="R9" gate="G$1" pin="1"/>
-<wire x1="43.18" y1="172.72" x2="58.42" y2="172.72" width="0.1524" layer="91"/>
+<wire x1="111.76" y1="157.48" x2="127" y2="157.48" width="0.1524" layer="91"/>
 <pinref part="R8" gate="G$1" pin="2"/>
-<wire x1="40.64" y1="172.72" x2="43.18" y2="172.72" width="0.1524" layer="91"/>
-<junction x="43.18" y="172.72"/>
+<wire x1="109.22" y1="157.48" x2="111.76" y2="157.48" width="0.1524" layer="91"/>
+<junction x="111.76" y="157.48"/>
 </segment>
 </net>
@@
 <segment>
 <pinref part="D1" gate="G$1" pin="AN"/>
-<wire x1="12.7" y1="134.62" x2="12.7" y2="132.08" width="0.1524" layer="91"/>
-<wire x1="12.7" y1="132.08" x2="25.4" y2="132.08" width="0.1524" layer="91"/>
-<wire x1="25.4" y1="132.08" x2="25.4" y2="127" width="0.1524" layer="91"/>
-<pinref part="U$3" gate="G$1" pin="1"/>
-<wire x1="25.4" y1="127" x2="22.86" y2="127" width="0.1524" layer="91"/>
-<label x="17.78" y="132.08" size="1.778" layer="95"/>
-</segment>
-</net>
+<wire x1="50.8" y1="116.84" x2="50.8" y2="111.76" width="0.1524" layer="91"/>
+<label x="43.18" y="111.76" size="1.778" layer="95"/>
+<pinref part="U$3" gate="G$1" pin="4"/>
+<wire x1="22.86" y1="111.76" x2="50.8" y2="111.76" width="0.1524" layer="91"/>
+</segment>
+</net>
