File: old/motherboard.brd (EAGLE design)
At the start: 71.1 x 35.6 mm, 34 parts

Commit message: started work on revised board
Parts:
- removed MICRO-USB: ZX80-B-5P, CUSTOM:USB_VERT
- removed U$1: BOURNS_4PIN, CUSTOM:BOURNS_4PIN
- added CONN: AVX_CONN, CUSTOM:AVX_CONN
- added USB: (no value), MicroUSB:USB-MICRO-SMD
Connections:
- net D+: now also USB.D+1; no longer MICRO-USB.D+
- net D-: now also USB.D-1; no longer MICRO-USB.D-
- net GND: now also CONN.P3, USB.G1, USB.G2, USB.G3, USB.G4, USB.G5, USB.G6, USB.GND1; no longer MICRO-USB.GND, MICRO-USB.GND1, MICRO-USB.GND2, MICRO-USB.GND3, MICRO-USB.GND4, U$1.P1, U$1.P3
- net N$3: now also USB.VBUS1; no longer MICRO-USB.VCC
- net N$5: now also CONN.P2; no longer U$1.P4
- net VCC: now also CONN.P1; no longer U$1.P2
Routing:
- net RST: track 67.6 -> 65.4 mm
- net D+: track 4.45 -> 6.19 mm
- net N$5: track 15.7 -> 17.2 mm
- net VCC: track 98.1 -> 99.1 mm
